File: kicad/VL53L5CX_Arduino_Shield/VL53L5CX_Arduino_Shield.kicad_sch (KiCad schematic)
At the start: 6 parts, among them J1 Conn_01x08_Pin, J2 Conn_01x05_Pin, J3 Conn_01x10_Pin, J4 Conn_01x08_Pin, J5 Conn_01x06_Socket, SW1 SW_MEC_5E

Commit message: Update schematic
Parts:
- added D1, D2: LED, symbol Device:LED
- added J6: Conn_01x05_Socket, symbol Connector:Conn_01x05_Socket
- added R1, R2: 1k, symbol Device:R
Connections:
- net GND: now also D1.1 (K), D2.1 (K)
- net at SW1.2: now also J1.3 (Pin_3); no longer J1.1 (Pin_1)
- net at J4.2 (Pin_2): now also R1.1
- net at J4.3 (Pin_3): now also R2.1
- net at J1.4 (Pin_4): now also J6.1 (Pin_1)
- net at J1.6 (Pin_6), J5.2 (Pin_2): now also J6.2 (Pin_2)
- net at J3.1 (Pin_1), J5.3 (Pin_3): now also J6.5 (Pin_5)
- net at J3.2 (Pin_2), J5.4 (Pin_4): now also J6.4 (Pin_4)
- new net: D2.2 (A), R2.2
- new net: D1.2 (A), R1.2
- no-connect marks 27 -> 26
Other:
- note added: "AMG8833 Module"
- note added: "D5"
- note added: "D6"
- note added: "ID4"
- note added: "VL53L5CX Module"
- moved on the sheet: J2, J4, SW1

Commit message: PointCloud 3D Viewer
Connections:
- net at J1.4 (Pin_4), J6.1 (Pin_1): now also J5.1 (Pin_1)
- net at J1.5 (Pin_5): no longer J5.1 (Pin_1)
Changed lines of the file:
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@@
 		(color 0 0 0 0)
 	)
+	(junction
+		(at 133.35 82.55)
+		(diameter 0)
+		(color 0 0 0 0)
+	)
 	(no_connect
 		(at 190.5 97.79)
@@
 	(wire
 		(pts
-			(xy 88.9 82.55) (xy 162.56 82.55)
+			(xy 88.9 82.55) (xy 133.35 82.55)
 		)
 		(stroke
@@
 	(wire
 		(pts
-			(xy 133.35 85.09) (xy 133.35 63.5)
-		)
-		(stroke
-			(width 0)
-			(type default)
-		)
-	)
-	(wire
-		(pts
 			(xy 115.57 59.69) (xy 121.92 59.69)
 		)
@@
 	(wire
 		(pts
-			(xy 88.9 85.09) (xy 133.35 85.09)
-		)
-		(stroke
-			(width 0)
-			(type default)
-		)
-	)
-	(wire
-		(pts
 			(xy 167.64 129.54) (xy 190.5 129.54)
 		)
@@
 	(wire
 		(pts
+			(xy 133.35 63.5) (xy 133.35 82.55)
+		)
+		(stroke
+			(width 0)
+			(type default)
+		)
+	)
+	(wire
+		(pts
 			(xy 170.18 63.5) (xy 170.18 77.47)
 		)
@@
 		)
 		(stroke
+			(width 0)
+			(type default)
+		)
+	)
+	(wire
+		(pts
+			(xy 133.35 82.55) (xy 162.56 82.55)
+		)
+		(stroke

Commit message: Schematic update
Connections:
- net GND: now also R1.2; no longer D1.1 (K)
- net at J4.2 (Pin_2): now also D1.2 (A); no longer R1.1
- new net: D1.1 (K), R1.1
Other:
- moved on the sheet: D1, R1
Changed lines of the file:
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@@
+	)
+	(junction
+		(at 170.18 77.47)
+		(diameter 0)
+		(color 0 0 0 0)
 	)
 	(junction
@@
 	)
 	(junction
-		(at 170.18 77.47)
-		(diameter 0)
-		(color 0 0 0 0)
-	)
-	(junction
 		(at 172.72 74.93)
 		(diameter 0)
@@
 	(wire
 		(pts
+			(xy 140.97 127) (xy 140.97 132.08)
+		)
+		(stroke
+			(width 0)
+			(type default)
+		)
+	)
+	(wire
+		(pts
 			(xy 140.97 139.7) (xy 140.97 143.51)
 		)
@@
 	(wire
 		(pts
+			(xy 97.79 80.01) (xy 97.79 59.69)
+		)
+		(stroke
+			(width 0)
+			(type default)
+		)
+	)
+	(wire
+		(pts
+			(xy 165.1 87.63) (xy 135.89 87.63)
+		)
+		(stroke
+			(width 0)
+			(type default)
+		)
+	)
+	(wire
+		(pts
+			(xy 140.97 160.02) (xy 140.97 163.83)
+		)
+		(stroke
+			(width 0)
+			(type default)
+		)
+	)
+	(wire
+		(pts
+			(xy 140.97 160.02) (xy 167.64 160.02)
+		)
+		(stroke
+			(width 0)
+			(type default)
+		)
+	)
+	(wire
+		(pts
+			(xy 172.72 63.5) (xy 172.72 74.93)
+		)
+		(stroke
+			(width 0)
+			(type default)
+		)
+	)
+	(wire
+		(pts
+			(xy 115.57 59.69) (xy 121.92 59.69)
+		)
+		(stroke
+			(width 0)
+			(type default)
+		)
+	)
+	(wire
+		(pts
+			(xy 135.89 87.63) (xy 135.89 63.5)
+		)
+		(stroke
+			(width 0)
+			(type default)
+		)
+	)
+	(wire
+		(pts
+			(xy 190.5 74.93) (xy 172.72 74.93)
+		)
+		(stroke
+			(width 0)
+			(type default)
+		)
+	)
+	(wire
+		(pts
 			(xy 140.97 151.13) (xy 140.97 160.02)
 		)
@@
 	(wire
 		(pts
-			(xy 97.79 80.01) (xy 97.79 59.69)
-		)
-		(stroke
-			(width 0)
-			(type default)
-		)
-	)
-	(wire
-		(pts
-			(xy 165.1 87.63) (xy 135.89 87.63)
-		)
-		(stroke
-			(width 0)
-			(type default)
-		)
-	)
-	(wire
-		(pts
-			(xy 140.97 160.02) (xy 140.97 163.83)
-		)
-		(stroke
-			(width 0)
-			(type default)
-		)
-	)
-	(wire
-		(pts
-			(xy 172.72 63.5) (xy 172.72 74.93)
-		)
-		(stroke
-			(width 0)
-			(type default)
-		)
-	)
-	(wire
-		(pts
-			(xy 115.57 59.69) (xy 121.92 59.69)
-		)
-		(stroke
-			(width 0)
-			(type default)
-		)
-	)
-	(wire
-		(pts
-			(xy 135.89 87.63) (xy 135.89 63.5)
-		)
-		(stroke
-			(width 0)
-			(type default)
-		)
-	)
-	(wire
-		(pts
-			(xy 140.97 160.02) (xy 167.64 160.02)
-		)
-		(stroke
-			(width 0)
-			(type default)
-		)
-	)
-	(wire
-		(pts
-			(xy 190.5 74.93) (xy 172.72 74.93)
-		)
-		(stroke
-			(width 0)
-			(type default)
-		)
-	)
-	(wire
-		(pts
 			(xy 167.64 129.54) (xy 190.5 129.54)
 		)
@@
 		(pts
 			(xy 167.64 139.7) (xy 167.64 143.51)
-		)
-		(stroke
-			(width 0)
-			(type default)
-		)
-	)
-	(wire
-		(pts
-			(xy 140.97 127) (xy 140.97 132.08)
 		)
 		(stroke
@@
 	(symbol
 		(lib_id "Device:R")
-		(at 140.97 135.89 0)
+		(at 140.97 147.32 0)
 		(unit 1)
 		(body_style 1)
@@
 		(fields_autoplaced yes)
 		(property "Reference" "R1"
-			(at 143.51 134.6199 0)
+			(at 143.51 146.0499 0)
 			(show_name no)
 			(do_not_autoplace no)
@@
 		)
 		(property "Value" "1k"
-			(at 143.51 137.1599 0)
+			(at 143.51 148.5899 0)
 			(show_name no)
 			(do_not_autoplace no)
@@
 		)
 		(property "Footprint" ""
-			(at 139.192 135.89 90)
+			(at 139.192 147.32 90)
 			(hide yes)
 			(show_name no)
@@
 		)
 		(property "Datasheet" ""
-			(at 140.97 135.89 0)
+			(at 140.97 147.32 0)
 			(hide yes)
 			(show_name no)
@@
 		)
 		(property "Description" "Resistor"
-			(at 140.97 135.89 0)
+			(at 140.97 147.32 0)
 			(hide yes)
 			(show_name no)
@@
 	(symbol
 		(lib_id "Device:LED")
-		(at 140.97 147.32 90)
+		(at 140.97 135.89 90)
 		(unit 1)
 		(body_style 1)
@@
 		(fields_autoplaced yes)
 		(property "Reference" "D1"
-			(at 144.78 147.6374 90)
+			(at 144.78 136.2074 90)
 			(show_name no)
 			(do_not_autoplace no)
@@
 		)
 		(property "Value" "LED"
-			(at 144.78 150.1774 90)
+			(at 144.78 138.7474 90)
 			(show_name no)
 			(do_not_autoplace no)
@@
 		)
 		(property "Footprint" ""
-			(at 140.97 147.32 0)
+			(at 140.97 135.89 0)
 			(hide yes)
 			(show_name no)
@@
 		)
 		(property "Datasheet" ""
-			(at 140.97 147.32 0)
+			(at 140.97 135.89 0)
 			(hide yes)
 			(show_name no)
@@
 		)
 		(property "Description" "Light emitting diode"
-			(at 140.97 147.32 0)
+			(at 140.97 135.89 0)
 			(hide yes)
 			(show_name no)
@@
 		)
 		(property "Sim.Pins" "1=K 2=A"
-			(at 140.97 147.32 0)
-			(hide yes)
-			(show_name no)
+			(at 140.97 135.89 0)
+			(hide yes)
+			(show_name no)
